File: x6-pcb.sch (KiCad schematic (older format))
At the start: 28 parts, among them SW1 SW_Push, U1 ATmega32U4-AU, Y1 16MHz

Commit message: Removed switch LEDs
Parts:
- MX1, MX2, MX3, MX4, MX5, MX6: footprint MX_Only:MXOnly-1U -> MX_Only:MXOnly-1U-NoLED
Changed lines of the file:
@@
 F 0 "MX1" H 7483 3723 60  0000 C CNN
 F 1 "MX-NoLED" H 7483 3649 20  0000 C CNN
-F 2 "MX_Only:MXOnly-1U" H 6825 3475 60  0001 C CNN
+F 2 "MX_Only:MXOnly-1U-NoLED" H 6825 3475 60  0001 C CNN
 F 3 "" H 6825 3475 60  0001 C CNN
 	1    7450 3500
@@
 F 0 "MX2" H 7983 3723 60  0000 C CNN
 F 1 "MX-NoLED" H 7983 3649 20  0000 C CNN
-F 2 "MX_Only:MXOnly-1U" H 7325 3475 60  0001 C CNN
+F 2 "MX_Only:MXOnly-1U-NoLED" H 7325 3475 60  0001 C CNN
 F 3 "" H 7325 3475 60  0001 C CNN
 	1    7950 3500
@@
 F 0 "MX3" H 8483 3723 60  0000 C CNN
 F 1 "MX-NoLED" H 8483 3649 20  0000 C CNN
-F 2 "MX_Only:MXOnly-1U" H 7825 3475 60  0001 C CNN
+F 2 "MX_Only:MXOnly-1U-NoLED" H 7825 3475 60  0001 C CNN
 F 3 "" H 7825 3475 60  0001 C CNN
 	1    8450 3500
@@
 F 0 "MX4" H 7483 4373 60  0000 C CNN
 F 1 "MX-NoLED" H 7483 4299 20  0000 C CNN
-F 2 "MX_Only:MXOnly-1U" H 6825 4125 60  0001 C CNN
+F 2 "MX_Only:MXOnly-1U-NoLED" H 6825 4125 60  0001 C CNN
 F 3 "" H 6825 4125 60  0001 C CNN
 	1    7450 4150
@@
 F 0 "MX5" H 7983 4373 60  0000 C CNN
 F 1 "MX-NoLED" H 7983 4299 20  0000 C CNN
-F 2 "MX_Only:MXOnly-1U" H 7325 4125 60  0001 C CNN
+F 2 "MX_Only:MXOnly-1U-NoLED" H 7325 4125 60  0001 C CNN
 F 3 "" H 7325 4125 60  0001 C CNN
 	1    7950 4150
@@
 F 0 "MX6" H 8483 4373 60  0000 C CNN
 F 1 "MX-NoLED" H 8483 4299 20  0000 C CNN
-F 2 "MX_Only:MXOnly-1U" H 7825 4125 60  0001 C CNN
+F 2 "MX_Only:MXOnly-1U-NoLED" H 7825 4125 60  0001 C CNN
 F 3 "" H 7825 4125 60  0001 C CNN
 	1    8450 4150
